File: kicad/apple2-luggable-crt.kicad_pcb (KiCad board)
At the start: 2 copper layers, 169 parts, among them J401 DEFLECTION YOKE, J801 12V UNREG, Q402 2SC2233, Q501 TD7698AP, SW201 SW_SP3T, T401 L_Ferrite_Coupled_1243, T451 KFB-2007 / 8D04K, T502 KRFE204, X501 3.579545MHz

Commit message: more progress
Parts:
- added C201: 33μF 16V, Capacitor_THT:CP_Radial_D5.0mm_P2.00mm, F.Cu at (162.0, 58.1)
- added C204: 330μF 16V, Capacitor_THT:CP_Radial_D8.0mm_P3.50mm, F.Cu at (143.0, 28.5)
- added C205: 1μF 50V, Capacitor_SMD:C_0805_2012Metric_Pad1.18x1.45mm_HandSolder, F.Cu at (162.1, 44.3)
- added C208: 10μF 50V, Capacitor_SMD:C_0805_2012Metric_Pad1.18x1.45mm_HandSolder, F.Cu at (162.1, 47.3)
- added C209: 220μF 16V, Capacitor_THT:CP_Radial_D8.0mm_P3.50mm, F.Cu at (143.0, 38.0)
- added C210: 1000μF 16V, Capacitor_THT:CP_Radial_D8.0mm_P3.50mm, F.Cu at (152.8, 28.5)
- added C303: 0.47μF 50V BP, Capacitor_SMD:C_0805_2012Metric_Pad1.18x1.45mm_HandSolder, F.Cu at (162.1, 50.3)
- added C305: 2.2μF 25V, Capacitor_SMD:C_0805_2012Metric_Pad1.18x1.45mm_HandSolder, F.Cu at (162.1, 53.3)
- added C306: 100μF 25V, Capacitor_THT:CP_Radial_D6.3mm_P2.50mm, F.Cu at (154.5, 46.7)
- added C308: 1μF 25V, Capacitor_SMD:C_0805_2012Metric_Pad1.18x1.45mm_HandSolder, F.Cu at (166.9, 44.3)
- added C309: 1000μF 16V, Capacitor_THT:CP_Radial_D8.0mm_P3.50mm, F.Cu at (152.8, 38.0)
- added C310: 1000μF 16V, Capacitor_THT:CP_Radial_D8.0mm_P3.50mm, F.Cu at (162.5, 28.5)
- added C311: 0.1μF 50V, Capacitor_SMD:C_0805_2012Metric_Pad1.18x1.45mm_HandSolder, F.Cu at (166.9, 47.3)
- added C314: 1μF 25V, Capacitor_SMD:C_0805_2012Metric_Pad1.18x1.45mm_HandSolder, F.Cu at (166.9, 50.3)
- added C401: 1μF 50V, Capacitor_SMD:C_0805_2012Metric_Pad1.18x1.45mm_HandSolder, F.Cu at (166.9, 53.3)
- added C408: 1μF 50V, Capacitor_SMD:C_0805_2012Metric_Pad1.18x1.45mm_HandSolder, F.Cu at (171.7, 44.3)
- added C409: 1μF 50V, Capacitor_SMD:C_0805_2012Metric_Pad1.18x1.45mm_HandSolder, F.Cu at (171.7, 47.3)
- added C412: 220μF 16V, Capacitor_THT:CP_Radial_D8.0mm_P3.50mm, F.Cu at (162.5, 38.0)
- added C416: 0.47μF 50V BP, Capacitor_SMD:C_0805_2012Metric_Pad1.18x1.45mm_HandSolder, F.Cu at (171.7, 50.3)
- added C419: 22nF 200V, Capacitor_THT:C_Rect_L10.3mm_W4.5mm_P7.50mm_MKS4, F.Cu at (142.0, 45.8)
- added C420: 10nF 200V, Capacitor_THT:C_Rect_L10.3mm_W4.5mm_P7.50mm_MKS4, F.Cu at (142.0, 51.9)
- added C421: 27nF 200V, Capacitor_THT:C_Rect_L10.3mm_W4.5mm_P7.50mm_MKS4, F.Cu at (142.0, 57.9)
- added C422: 4.7μF 160V, Capacitor_THT:CP_Radial_D6.3mm_P2.50mm, F.Cu at (156.5, 68.0)
- added C423: 1000μF 16V, Capacitor_THT:CP_Radial_D8.0mm_P3.50mm, F.Cu at (172.3, 28.5)
- added C424: 100μF 25V, Capacitor_THT:CP_Radial_D6.3mm_P2.50mm, F.Cu at (154.5, 54.6)
- added C503: 1μF 50V, Capacitor_SMD:C_0805_2012Metric_Pad1.18x1.45mm_HandSolder, F.Cu at (171.7, 53.3)
- added C508: 0.47μF 50V, Capacitor_SMD:C_0805_2012Metric_Pad1.18x1.45mm_HandSolder, F.Cu at (164.1, 65.6)
- added C513: 4.7μF 50V, Capacitor_SMD:C_0805_2012Metric_Pad1.18x1.45mm_HandSolder, F.Cu at (164.1, 68.6)
- added C519: 51pF, Capacitor_SMD:C_0805_2012Metric_Pad1.18x1.45mm_HandSolder, F.Cu at (169.1, 58.4)
- added C803: 330μF 16V, Capacitor_THT:CP_Radial_D8.0mm_P3.50mm, F.Cu at (172.3, 38.0)
- added D202: 1N4148, Diode_SMD:D_MiniMELF_Handsoldering, F.Cu at (130.1, 78.2)
- added D203: 1N4148, Diode_SMD:D_MiniMELF_Handsoldering, F.Cu at (130.1, 81.6)
- added D301: 1N4148, Diode_SMD:D_MiniMELF_Handsoldering, F.Cu at (130.1, 84.9)
- added D302: 1N4148, Diode_SMD:D_MiniMELF_Handsoldering, F.Cu at (130.1, 88.3)
- added D303: 1N4935, Diode_THT:D_DO-41_SOD81_P10.16mm_Horizontal, F.Cu at (137.2, 78.7)
- added D401: 1N4148, Diode_SMD:D_MiniMELF_Handsoldering, F.Cu at (130.1, 91.6)
- added D402: 1N4148, Diode_SMD:D_MiniMELF_Handsoldering, F.Cu at (130.1, 94.9)
- added D403: 1N4148, Diode_SMD:D_MiniMELF_Handsoldering, F.Cu at (130.1, 98.3)
- added D404: 1N4935, Diode_THT:D_DO-41_SOD81_P10.16mm_Horizontal, F.Cu at (137.2, 82.9)
- added D405: ???, Diode_THT:D_DO-41_SOD81_P10.16mm_Horizontal, F.Cu at (137.2, 87.2)
- added D408: 1N4935, Diode_THT:D_DO-41_SOD81_P10.16mm_Horizontal, F.Cu at (137.2, 91.4)
- added J402: CRT SOCKET BRD, Connector_JST:JST_XH_B4B-XH-A_1x04_P2.50mm_Vertical, F.Cu at (127.1, 106.7)
- added J501: CRT SOCKET BRD, Connector_JST:JST_XH_B5B-XH-A_1x05_P2.50mm_Vertical, F.Cu at (142.4, 106.7)
- added L405: 10μH, foodprints:L_Radial_D10.0mm_P7.62mm, F.Cu at (29.2, 119.4)
- added Q201: 2SA562-Y, Package_TO_SOT_THT:TO-92_Inline_Wide, F.Cu at (152.4, 78.7)
- added Q202: 2SC1815-Y, Package_TO_SOT_THT:TO-92_Inline_Wide, F.Cu at (40.6, 119.1)
- added Q301: 2SC2236A-Y, Package_TO_SOT_THT:TO-92_Inline_Wide, F.Cu at (40.6, 124.9)
- added Q302: 2SC2236A-Y, Package_TO_SOT_THT:TO-92_Inline_Wide, F.Cu at (40.6, 130.7)
- added Q303: 2SC1815-Y, Package_TO_SOT_THT:TO-92_Inline_Wide, F.Cu at (40.6, 136.4)
- added Q304: 2SA1015-Y, Package_TO_SOT_THT:TO-92_Inline_Wide, F.Cu at (40.6, 142.2)
- added Q401: 2SC200-Y, Package_TO_SOT_THT:TO-92_Inline_Wide, F.Cu at (48.3, 142.2)
- L301: footprint Inductor_THT:L_Radial_D7.5mm_P5.00mm_Fastron_07P -> Inductor_SMD:L_1008_2520Metric_Pad1.43x2.20mm_HandSolder
- L408, L501: footprint Inductor_THT:L_Radial_D7.5mm_P5.00mm_Fastron_07P -> Inductor_SMD:L_TDK_NLV32_3.2x2.5mm
- R206: value 830Ω -> 820Ω
- R321: value 160Ω 1/2 W -> 160Ω 1/2W

Commit message: more work
Parts:
- added H1: MountingHole_Pad, MountingHole:MountingHole_3.2mm_M3_Pad_TopBottom, F.Cu at (26.0, 26.5)
- added H2: MountingHole_Pad, MountingHole:MountingHole_3.2mm_M3_Pad_TopBottom, F.Cu at (26.0, 104.3)
- added H3: MountingHole_Pad, MountingHole:MountingHole_3.2mm_M3_Pad_TopBottom, F.Cu at (194.1, 103.8)
- added H4: MountingHole_Pad, MountingHole:MountingHole_3.2mm_M3_Pad_TopBottom, F.Cu at (195.6, 24.0)
- added H5: MountingHole_Pad, MountingHole:MountingHole_3.2mm_M3_Pad_TopBottom, F.Cu at (193.4, 54.1)
- added H6: MountingHole_Pad, MountingHole:MountingHole_3.2mm_M3_Pad_TopBottom, F.Cu at (139.5, 34.9)
- added R254: 10kΩ B, Potentiometer_THT:Potentiometer_Alpha_RD901F-40-00D_Single_Vertical_CircularHoles, F.Cu at (227.4, 26.0)
- added R255: 10kΩ B, Potentiometer_THT:Potentiometer_Alpha_RD901F-40-00D_Single_Vertical_CircularHoles, F.Cu at (227.4, 40.4)
- added R257: 5kΩ, Potentiometer_THT:Potentiometer_Bourns_3386F_Vertical, F.Cu at (171.4, 132.2)
- added R352: 5kΩ B, Potentiometer_THT:Potentiometer_Bourns_3386F_Vertical, F.Cu at (182.4, 132.2)
- added R353: 470Ω B, Potentiometer_THT:Potentiometer_Bourns_3386F_Vertical, F.Cu at (193.5, 132.2)
- added R451: 10kΩ B, Potentiometer_THT:Potentiometer_Alpha_RD901F-40-00D_Single_Vertical_CircularHoles, F.Cu at (227.4, 54.8)
- added R554: 10kΩ B, Potentiometer_THT:Potentiometer_Alpha_RD901F-40-00D_Single_Vertical_CircularHoles, F.Cu at (227.4, 69.2)
- added R555: 10kΩ B, Potentiometer_THT:Potentiometer_Alpha_RD901F-40-00D_Single_Vertical_CircularHoles, F.Cu at (227.4, 83.6)
- C203, C205, C206, C207, C301, C302, C303, C304, C305, C307, C308, C311, C312, C314, C403, C404, C407, C413, C415, C427, C428, C430, C434, C501, C502, C503, C508, C509, C510, C511, C513, C516, C517, C518, C519, D302, D403, L301, L501, R204, R205, R206, R208, R209, R220, R223, R224, R227, R300, R301, R302, R303, R304, R313, R315, R316, R317, R323, R324, R325, R326, R327, R328, R329, R354, R355, R403, R404, R405, R410, R412, R413, R501, R502, R503, R511, R516, R517, R518, R520, R524, R525, R527, R529, R531, R535: moved to B.Cu
- moved Q401 352.0 mm to (134.6, -199.0)
- moved R306 316.4 mm to (362.4, -58.0)
- moved Q402 310.4 mm to (208.1, -194.2)
- moved T401 310.4 mm to (207.0, -183.0)
- moved R202 288.8 mm to (332.4, -21.4)
- moved R203 288.8 mm to (332.4, -18.1)
- moved C435 284.4 mm to (363.4, -64.0)
- moved R226 282.6 mm to (330.4, -10.0)
- moved L410 270.8 mm to (177.0, -173.0)
- moved RV14 268.2 mm to (340.4, -13.0)
- moved TP1 256.2 mm to (248.0, -183.0)
- moved C418 253.7 mm to (149.0, -197.7)
- moved C429 253.7 mm to (153.8, -206.8)
- moved C417 253.7 mm to (149.0, -200.8)
- moved C426 253.7 mm to (149.0, -194.7)
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Connections:
- C407 pad 1: Net-(Q501-H_OSC_TIMING) -> GNDPWR
- C407 pad 2: GNDPWR -> Net-(Q501-H_OSC_TIMING)
- L301 pad 1: Net-(Q501-SYNC_SEP._OUT) -> Net-(C301-Pad1)
- L301 pad 2: Net-(C301-Pad1) -> Net-(Q501-SYNC_SEP._OUT)
- R324 pad 1: Net-(C311-Pad2) -> Net-(Q303-B)
- R324 pad 2: Net-(Q303-B) -> Net-(C311-Pad2)
- R410 pad 1: Net-(Q501-H_OSC_TIMING) -> Net-(R410-Pad1)
- R410 pad 2: Net-(R410-Pad2) -> Net-(Q501-H_OSC_TIMING)
- R412 pad 1: Net-(Q501-H_OSC_TIMING) -> +VCC_{H}
- R412 pad 2: +VCC_{H} -> Net-(Q501-H_OSC_TIMING)
Routing:
- net Net-(D403-K): track 0.00 -> 85.6 mm
- net Net-(D408-K): track 0.00 -> 82.4 mm
- net Net-(D203-A): track 0.00 -> 69.9 mm
- net Net-(Q301-B): track 0.00 -> 66.6 mm
- net Net-(D405-K): track 0.00 -> 64.0 mm
- net Net-(C308-Pad1): track 0.00 -> 57.8 mm
- net Net-(Q501-V_OSC_TIMING): track 0.00 -> 48.0 mm
- net Net-(J401-Pin_3): track 0.00 -> 46.6 mm
- net +11V: track 0.00 -> 40.2 mm
- net Net-(Q501-CONTRAST_OUT_(C)): track 0.00 -> 36.2 mm
- net Net-(Q501-CHROMA_OUT): track 0.00 -> 32.8 mm
- net +VCC_{H}: track 0.00 -> 28.9 mm
- net Net-(Q202-B): track 0.00 -> 23.4 mm
- net Net-(D404-K): track 0.00 -> 23.4 mm
- net Net-(Q501-B-Y_OUT): track 0.00 -> 23.1 mm
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- added copper zone on F.Cu, net +10V
- added copper zone on F.Cu, net +11V
- added copper zone on B.Cu, net GNDPWR
Other:
- board outline added: 225 x 110 mm
