File: kicad/apple2-luggable-crt.kicad_pcb (KiCad board)
At the start: 2 copper layers, 225 x 110 mm, 234 parts, among them J401 DEFLECTION YOKE, J402 CRT SOCKET BRD, J501 CRT SOCKET BRD, J801 12V UNREG, Q201 2SA562-Y, Q202 2SC1815-Y, Q301 2SC2236A-Y, Q302 2SC2236A-Y, Q303 2SC1815-Y, Q304 2SA1015-Y, Q401 2SC200-Y, Q402 2SC2233, Q501 TD7698AP, SW201 SW_SP3T, T401 L_Ferrite_Coupled_1243, T451 KFB-2007 / 8D04K, T502 KRFE204, X501 3.579545MHz

Commit message: more progress
- pretty close to being done.  now comparing foot prints to parts samples, checking part placement for interference, and making layout adjustments to accommodate PCB mounting holes now that I know where they are.
Parts:
- removed C803: 330μF 16V, Capacitor_THT:CP_Radial_D8.0mm_P3.50mm
- added J1: VIDEO IN, Connector_Coaxial:BNC_TEConnectivity_1478204_Vertical, F.Cu at (71.9, 28.2)
- added J403: PICTURE CONTROLS, Connector_JST:JST_PH_B9B-PH-K_1x09_P2.00mm_Vertical, B.Cu at (77.5, 135.0)
- added J404: PICTURE CONTROLS, Connector_JST:JST_PH_B9B-PH-K_1x09_P2.00mm_Vertical, F.Cu at (81.6, 25.3)
- added R211: 6.81kΩ 1%, Resistor_SMD:R_1206_3216Metric_Pad1.30x1.75mm_HandSolder, F.Cu at (125.3, 34.5)
- added R212: 53.6kΩ 1%, Resistor_SMD:R_1206_3216Metric_Pad1.30x1.75mm_HandSolder, F.Cu at (125.3, 39.6)
- added R351: 200kΩ B, Potentiometer_THT:Potentiometer_Alpha_RD901F-40-00D_Single_Vertical_CircularHoles, F.Cu at (107.9, 130.6)
- added REF**: Heatsink_Fischer_FK224xx2201_25x8.3mm, Heatsink:Heatsink_Fischer_FK224xx2201_25x8.3mm, F.Cu at (126.6, 59.8)
- added U1: XRP29302ETBTR-L, Package_TO_SOT_SMD:TO-263-5_TabPin3, F.Cu at (117.4, 30.0)
- C202, C208, C210, C405, C414, C417, C418, C426, C429, C504, C506, D402, R203, R213, R214, R230, R257, R305, R406, R415, R417, R424, R426, R507, R515, R519, RV14: moved to B.Cu
- H1, H2, H3, H4, H5, H6: value MountingHole_Pad -> M3
- J801: footprint Connector_BarrelJack:BarrelJack_Wuerth_6941xx301002 -> TerminalBlock_TE-Connectivity:TerminalBlock_TE_282834-2_1x02_P2.54mm_Horizontal
- R355: moved to F.Cu
- moved C435 330.0 mm to (101.5, 136.7), turned to 180 degrees
- moved R306 321.7 mm to (106.4, 136.7), turned to 180 degrees
- moved Q401 285.0 mm to (139.8, 86.0), turned to 90 degrees
- moved C417 284.5 mm to (136.7, 83.4), turned to 180 degrees
- moved C418 277.7 mm to (149.8, 80.0)
- moved T401 273.9 mm to (143.7, 83.4)
- moved C201 272.2 mm to (75.8, 47.8), turned to 180 degrees
- moved RV14 272.0 mm to (74.7, 45.3)
- moved C426 271.2 mm to (147.2, 76.4), turned to 180 degrees
- moved R417 271.0 mm to (145.2, 80.0), turned to 180 degrees
- moved C429 270.0 mm to (139.6, 62.9)
- moved R202 268.7 mm to (74.7, 54.6), turned to 180 degrees
- moved R203 268.5 mm to (76.2, 61.9), turned to 90 degrees
- moved R226 263.2 mm to (74.7, 51.9)
- moved Q402 262.7 mm to (141.1, 59.8), turned to 180 degrees
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Connections:
- net Net-(Q501-BRIGHTNESS_CONTROL) renamed /BRIGHT
- net Net-(Q501-V_OSC_TIMING) renamed /V HOLD
- net Net-(R410-Pad1) renamed /H HOLD
- R230 pad 1: Net-(K6-A) -> Net-(R230-Pad1)
- R254 pad : (no net) -> GNDPWR
- R254 pad 1: Net-(R213-Pad1) -> Net-(R210-Pad2)
- R254 pad 3: Net-(R210-Pad2) -> Net-(R213-Pad1)
- R255 pad : (no net) -> GNDPWR
- R255 pad 1: Net-(R215-Pad2) -> Net-(R215-Pad1)
- R255 pad 3: Net-(R215-Pad1) -> Net-(R215-Pad2)
- R257 pad 3: Net-(K6-B) -> Net-(R230-Pad1)
- R451 pad : (no net) -> GNDPWR
- R451 pad 1: GNDPWR -> +VCC_{H}
- R451 pad 3: +VCC_{H} -> GNDPWR
- R554 pad : (no net) -> GNDPWR
- R554 pad 1: Net-(R515-Pad1) -> Net-(R512-Pad2)
- R554 pad 3: Net-(R512-Pad2) -> Net-(R515-Pad1)
- R555 pad : (no net) -> GNDPWR
- R555 pad 1: Net-(R507-Pad1) -> Net-(R504-Pad2)
- R555 pad 3: Net-(R504-Pad2) -> Net-(R507-Pad1)
Routing:
- net /CONTRAST: track 0.00 -> 139.7 mm
- net /COLOUR: track 0.00 -> 138.0 mm
- net /TINT: track 0.00 -> 123.2 mm
- net Net-(C208-Pad1): track 0.00 -> 117.4 mm
- net /V HOLD: track 48.0 -> 159.2 mm
- net Net-(R229-Pad2): track 0.00 -> 97.4 mm
- net /H HOLD: track 0.00 -> 89.9 mm
- net +VCC_{H}: track 28.9 -> 116.2 mm
- net /BRIGHT: track 3.06 -> 81.4 mm
- net Net-(R308-Pad2): track 0.00 -> 69.3 mm
- net Net-(D202-A): track 0.00 -> 52.5 mm
- net Net-(L407-Pad1): track 11.1 -> 50.3 mm
- net /H. PULSE: track 0.00 -> 34.8 mm
- net +11V: track 40.2 -> 6.42 mm
- net Net-(Q301-B): track 66.6 -> 89.1 mm
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- added copper zone on F.Cu, net GNDPWR
Other:
- board size 225 x 110 mm -> 145.3 x 120.3 mm

Commit message: version before heat sink work
Parts:
- added J2: FOC. SCN. RET., Connector_PinHeader_2.54mm:PinHeader_1x01_P2.54mm_Vertical, F.Cu at (136.2, 77.9)
- C507, R207, R215: moved to B.Cu
- H1, H2, H3, H4: value M3 -> M4; footprint MountingHole:MountingHole_3.2mm_M3_Pad_TopBottom -> MountingHole:MountingHole_4.3mm_M4_Pad_TopBottom
- H5, H6: footprint MountingHole:MountingHole_3.2mm_M3_Pad_TopBottom -> foodprints:MountingHole_3.2mm_M3_Pad_TopBottom_flyback_shield
- J801: footprint TerminalBlock_TE-Connectivity:TerminalBlock_TE_282834-2_1x02_P2.54mm_Horizontal -> Connector_JST:JST_VH_B2P-VH_1x02_P3.96mm_Vertical
- moved R230 86.3 mm to (104.4, 39.9), turned to 0 degrees
- moved C210 80.5 mm to (103.7, 55.9)
- moved J403 80.0 mm to (98.0, 57.6)
- moved R504 80.0 mm to (165.5, 58.2)
- moved R508 79.9 mm to (160.1, 58.2)
- moved R512 79.9 mm to (151.2, 58.2)
- moved R218 79.9 mm to (190.8, 58.2)
- moved R229 79.9 mm to (190.8, 41.2)
- moved R257 79.8 mm to (107.9, 43.8)
- moved C435 79.6 mm to (114.9, 58.2)
- moved R306 79.6 mm to (119.7, 58.2)
- moved R213 79.6 mm to (174.6, 48.6)
- moved R214 79.6 mm to (176.7, 55.5)
- moved R507 79.6 mm to (160.6, 48.7)
- moved R515 79.6 mm to (146.4, 48.6)
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- renumbered RV14 to R129
Connections:
- net Net-(D405-K) renamed /90V
- net Net-(J402-Pin_1) renamed /HEATER ACV
- net Net-(J801-Pin_1) renamed /12 V UNREG
Routing:
- net Net-(D202-A): track 52.5 -> 2.55 mm
- net Net-(J2-Pin_1): track 18.7 -> 65.1 mm
- net Net-(R308-Pad2): track 69.3 -> 38.3 mm
- net Net-(C310-Pad2): track 19.7 -> 46.2 mm
- net Net-(C209-Pad1): track 10.4 -> 34.5 mm
- net /VERT BLANKING: track 28.9 -> 10.3 mm
- net /V HOLD: track 159.2 -> 145.5 mm
- net /H. PULSE: track 34.8 -> 46.8 mm
- net Net-(R352-Pad3): track 10.2 -> 20.5 mm
- net Net-(R215-Pad1): track 19.4 -> 9.22 mm
- net Net-(Q202-B): track 24.1 -> 14.1 mm
- net /BRIGHT: track 81.4 -> 90.8 mm
- net Net-(C308-Pad1): track 77.7 -> 87.0 mm
- net Net-(C208-Pad1): track 117.4 -> 109.1 mm
- net Net-(L406-Pad1): track 15.2 -> 7.19 mm
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Other:
- board size 145.3 x 120.3 mm -> 145.3 x 115.9 mm
- board text added: "https://github.com/cannon-zz/luggable-colour-crt-monitor.git"

Commit message: finished.
Parts:
- removed REF**: Heatsink_Fischer_FK224xx2201_25x8.3mm, Heatsink:Heatsink_Fischer_FK224xx2201_25x8.3mm
- added HS1: Heatsink_Pad_2Pin, foodprints:Heatsink_TO-220_26x20mm_2xFixation1.2mm, F.Cu at (124.5, 100.4)
- R319: moved to B.Cu
- moved C419 44.2 mm to (158.5, 116.2), turned to 0 degrees
- moved D408 18.3 mm to (137.0, 106.2), turned to -90 degrees
- moved J404 16.4 mm to (59.3, 68.7)
- moved L409 13.4 mm to (123.9, 85.2), turned to 90 degrees
- moved R312 11.2 mm to (148.8, 129.5), turned to 0 degrees
- moved J1 10.6 mm to (60.8, 82.2)
- moved R414 10.3 mm to (84.0, 94.1)
- moved R225 10.2 mm to (83.3, 90.3)
- moved R319 9.52 mm to (173.2, 118.0), turned to 180 degrees
- moved D202 9.02 mm to (91.8, 90.3)
- moved TP1 8.14 mm to (114.0, 69.0)
- moved U1 7.11 mm to (104.4, 73.7)
- moved J801 7.11 mm to (90.7, 68.9)
- moved R211 7.11 mm to (112.3, 78.2)
- moved R212 7.11 mm to (112.3, 83.3)
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Routing:
- net Net-(J401-Pin_3): track 53.6 -> 65.8 mm
- net /H HOLD: track 88.7 -> 78.4 mm
- net /COLOUR: track 141.6 -> 131.3 mm
- net Net-(D408-K): track 75.7 -> 65.7 mm
- net /V HOLD: track 145.5 -> 154.9 mm
- net Net-(J1-In): track 21.6 -> 12.8 mm
- net Net-(Q402-B): track 19.6 -> 27.5 mm
- net /TINT: track 124.7 -> 117.4 mm
- net Net-(Q402-E): track 9.29 -> 15.6 mm
- net +VCC_{H}: track 115.2 -> 109.8 mm
- net /CONTRAST: track 135.5 -> 130.7 mm
- net /BRIGHT: track 90.8 -> 86.6 mm
- net Net-(J2-Pin_1): track 65.1 -> 60.9 mm
- net Net-(C426-Pad1): track 10.0 -> 12.7 mm
- net Net-(D202-K): track 5.69 -> 8.38 mm
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
Commit message: add REV A to boards
Other:
- board text added: "REV A"
Changed lines of the file:
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@@
 	)
 	(gr_text "https://github.com/cannon-zz/luggable-colour-crt-monitor.git"
-		(at 122.287616 152.512988 0)
+		(at 130.155159 152.111993 0)
 		(layer "B.SilkS")
 		(effects
@@
 		)
 	)
+	(gr_text "REV A"
+		(at 91.039159 152.111993 0)
+		(layer "B.SilkS")
+		(effects
+			(font
+				(size 2 2)
+				(thickness 0.4)
+				(bold yes)
+			)
+			(justify left bottom mirror)
+		)
+	)
+	(gr_text "REV A"
+		(at 132.695159 59.655993 0)
+		(layer "B.SilkS")
+		(effects
+			(font
+				(size 2 2)
+				(thickness 0.4)
+				(bold yes)
+			)
+			(justify left bottom mirror)
+		)
+	)
