File: kicad/apple2-luggable-crt.kicad_pcb (KiCad board)
At the start: 2 copper layers, 145.3 x 115.9 mm, 242 parts, among them J1 VIDEO IN, J2 FOC. SCN. RET., J401 DEFLECTION YOKE, J402 CRT SOCKET BRD, J403 PICTURE CONTROLS, J404 PICTURE CONTROLS, J501 CRT SOCKET BRD, J801 12V UNREG, Q201 2SA562-Y, Q202 2SC1815-Y, Q301 2SC2236A-Y, Q302 2SC2236A-Y, Q303 2SC1815-Y, Q304 2SA1015-Y, Q401 2SC200-Y, Q402 2SC2233, Q501 TD7698AP, SW201 SW_SP3T, T401 L_Ferrite_Coupled_1243, T451 KFB-2007 / 8D04K, T502 KRFE204, U1 XRP29302ETBTR-L, X501 3.579545MHz

Commit message: some tweaks
Routing:
- net Net-(Q301-B): track 94.2 -> 97.5 mm
Changed lines of the file:
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@@
 			(sketchdnponfab yes)
 			(crossoutdnponfab yes)
-			(subtractmaskfromsilk no)
+			(subtractmaskfromsilk yes)
 			(outputformat 1)
 			(mirror no)
@@
 		)
 		(property "Value" "FOC. SCN. RET."
-			(at -7.747 0.879192 0)
+			(at 0.091 2.592005 0)
 			(layer "F.SilkS")
 			(effects
@@
 	)
 	(segment
-		(start 174.782462 132.879163)
-		(end 174.782462 122.05218)
-		(width 1.25)
-		(layer "F.Cu")
-		(net "Net-(J401-Pin_3)")
-	)
-	(segment
-		(start 171.597159 136.064466)
-		(end 174.782462 132.879163)
-		(width 1.25)
-		(layer "F.Cu")
-		(net "Net-(J401-Pin_3)")
-	)
-	(segment
-		(start 164.953159 136.064466)
-		(end 162.966686 134.077993)
-		(width 1.25)
-		(layer "F.Cu")
-		(net "Net-(J401-Pin_3)")
-	)
-	(segment
-		(start 164.953159 136.064466)
-		(end 171.597159 136.064466)
-		(width 1.25)
-		(layer "F.Cu")
-		(net "Net-(J401-Pin_3)")
-	)
-	(segment
-		(start 162.966686 134.077993)
-		(end 161.143159 134.077993)
-		(width 1.25)
-		(layer "F.Cu")
-		(net "Net-(J401-Pin_3)")
-	)
-	(segment
-		(start 164.953159 141.525466)
-		(end 164.953159 136.064466)
-		(width 1.25)
-		(layer "F.Cu")
-		(net "Net-(J401-Pin_3)")
-	)
-	(segment
-		(start 160.681445 145.79718)
-		(end 150.491183 145.79718)
-		(width 0.5)
-		(layer "B.Cu")
-		(net "Net-(J401-Pin_3)")
-	)
-	(segment
-		(start 150.491183 145.79718)
-		(end 149.592491 144.898488)
-		(width 0.5)
-		(layer "B.Cu")
-		(net "Net-(J401-Pin_3)")
-	)
-	(segment
-		(start 154.889873 132.85918)
-		(end 159.708252 132.85918)
-		(width 0.5)
-		(layer "B.Cu")
-		(net "Net-(J401-Pin_3)")
-	)
-	(segment
-		(start 174.782462 126.16518)
-		(end 174.782462 117.98818)
-		(width 1.25)
-		(layer "B.Cu")
-		(net "Net-(J401-Pin_3)")
-	)
-	(segment
-		(start 164.953159 141.525466)
-		(end 160.681445 145.79718)
-		(width 0.5)
-		(layer "B.Cu")
-		(net "Net-(J401-Pin_3)")
-	)
-	(segment
-		(start 159.708252 132.85918)
-		(end 160.927065 134.077993)
-		(width 0.5)
-		(layer "B.Cu")
-		(net "Net-(J401-Pin_3)")
-	)
-	(segment
-		(start 149.592491 144.898488)
-		(end 148.084616 144.898488)
-		(width 0.5)
-		(layer "B.Cu")
-		(net "Net-(J401-Pin_3)")
-	)
-	(segment
-		(start 169.782462 122.22418)
-		(end 172.707462 125.14918)
-		(width 1.25)
-		(layer "B.Cu")
-		(net "Net-(J401-Pin_2)")
-	)
-	(segment
-		(start 171.682462 117.98818)
-		(end 171.682462 120.15218)
-		(width 1.25)
-		(layer "B.Cu")
-		(net "Net-(J401-Pin_2)")
-	)
-	(segment
-		(start 172.707462 125.14918)
-		(end 172.707462 126.38218)
-		(width 1.25)
-		(layer "B.Cu")
-		(net "Net-(J401-Pin_2)")
-	)
-	(segment
-		(start 172.700159 142.110466)
-		(end 176.256159 145.666466)
-		(width 1.25)
-		(layer "B.Cu")
-		(net "Net-(J401-Pin_2)")
-	)
-	(segment
-		(start 172.707462 126.59918)
-		(end 172.707462 139.062466)
-		(width 1.25)
-		(layer "B.Cu")
-		(net "Net-(J401-Pin_2)")
-	)
-	(segment
-		(start 171.682462 120.15218)
-		(end 169.782462 122.05218)
-		(width 1.25)
-		(layer "B.Cu")
-		(net "Net-(J401-Pin_2)")
-	)
-	(segment
-		(start 172.700159 139.069769)
-		(end 172.700159 142.110466)
-		(width 1.25)
-		(layer "B.Cu")
-		(net "Net-(J401-Pin_2)")
-	)
-	(segment
-		(start 169.782462 122.05218)
-		(end 169.782462 122.22418)
-		(width 1.25)
-		(layer "B.Cu")
-		(net "Net-(J401-Pin_2)")
-	)
-	(segment
-		(start 172.707462 138.089163)
-		(end 172.707462 139.062466)
-		(width 1.25)
-		(layer "B.Cu")
-		(net "Net-(J401-Pin_2)")
-	)
-	(segment
 		(start 102.729616 108.852988)
 		(end 102.729616 105.804988)
@@
 	)
 	(segment
-		(start 143.488616 141.68018)
-		(end 130.560616 141.68018)
+		(start 141.339346 141.70618)
+		(end 130.534616 141.70618)
 		(width 0.5)
 		(layer "F.Cu")
@@
 	)
 	(segment
-		(start 159.923159 143.380466)
-		(end 145.188902 143.380466)
+		(start 162.286159 141.017466)
+		(end 152.171686 141.017466)
 		(width 0.5)
 		(layer "F.Cu")
@@
 	)
 	(segment
-		(start 162.286159 141.017466)
-		(end 159.923159 143.380466)
+		(start 143.555159 143.921993)
+		(end 141.339346 141.70618)
 		(width 0.5)
 		(layer "F.Cu")
@@
 	)
 	(segment
-		(start 130.560616 141.68018)
-		(end 130.534616 141.70618)
+		(start 152.171686 141.017466)
+		(end 149.267159 143.921993)
 		(width 0.5)
 		(layer "F.Cu")
@@
 	)
 	(segment
-		(start 145.188902 143.380466)
-		(end 143.488616 141.68018)
+		(start 149.267159 143.921993)
+		(end 143.555159 143.921993)
 		(width 0.5)
 		(layer "F.Cu")
@@
 	)
 	(segment
+		(start 174.782462 132.879163)
+		(end 174.782462 122.05218)
+		(width 1.25)
+		(layer "F.Cu")
+		(net "Net-(J401-Pin_3)")
+	)
+	(segment
+		(start 171.597159 136.064466)
+		(end 174.782462 132.879163)
+		(width 1.25)
+		(layer "F.Cu")
+		(net "Net-(J401-Pin_3)")
+	)
+	(segment
+		(start 164.953159 136.064466)
+		(end 162.966686 134.077993)
+		(width 1.25)
+		(layer "F.Cu")
+		(net "Net-(J401-Pin_3)")
+	)
+	(segment
+		(start 164.953159 136.064466)
+		(end 171.597159 136.064466)
+		(width 1.25)
+		(layer "F.Cu")
+		(net "Net-(J401-Pin_3)")
+	)
+	(segment
+		(start 162.966686 134.077993)
+		(end 161.143159 134.077993)
+		(width 1.25)
+		(layer "F.Cu")
+		(net "Net-(J401-Pin_3)")
+	)
+	(segment
+		(start 164.953159 141.525466)
+		(end 164.953159 136.064466)
+		(width 1.25)
+		(layer "F.Cu")
+		(net "Net-(J401-Pin_3)")
+	)
+	(segment
+		(start 160.681445 145.79718)
+		(end 150.491183 145.79718)
+		(width 0.5)
+		(layer "B.Cu")
+		(net "Net-(J401-Pin_3)")
+	)
+	(segment
+		(start 150.491183 145.79718)
+		(end 149.592491 144.898488)
+		(width 0.5)
+		(layer "B.Cu")
+		(net "Net-(J401-Pin_3)")
+	)
+	(segment
+		(start 154.889873 132.85918)
+		(end 159.708252 132.85918)
+		(width 0.5)
+		(layer "B.Cu")
+		(net "Net-(J401-Pin_3)")
+	)
+	(segment
+		(start 174.782462 126.16518)
+		(end 174.782462 117.98818)
+		(width 1.25)
+		(layer "B.Cu")
+		(net "Net-(J401-Pin_3)")
+	)
+	(segment
+		(start 164.953159 141.525466)
+		(end 160.681445 145.79718)
+		(width 0.5)
+		(layer "B.Cu")
+		(net "Net-(J401-Pin_3)")
+	)
+	(segment
+		(start 159.708252 132.85918)
+		(end 160.927065 134.077993)
+		(width 0.5)
+		(layer "B.Cu")
+		(net "Net-(J401-Pin_3)")
+	)
+	(segment
+		(start 149.592491 144.898488)
+		(end 148.084616 144.898488)
+		(width 0.5)
+		(layer "B.Cu")
+		(net "Net-(J401-Pin_3)")
+	)
+	(segment
 		(start 54.469616 124.092988)
 		(end 54.469616 121.070988)
@@
 	)
 	(segment
-		(start 169.398159 133.061993)
-		(end 163.470966 133.061993)
+		(start 163.216966 132.807993)
+		(end 159.391209 132.807993)
 		(width 0.5)
 		(layer "F.Cu")
@@
 	)
 	(segment
-		(start 110.501159 115.816179)
-		(end 110.501159 107.013567)
+		(start 159.391209 132.807993)
+		(end 148.977209 143.221993)
 		(width 0.5)
 		(layer "F.Cu")
@@
 	)
 	(segment
-		(start 163.470966 133.061993)
-		(end 163.216966 132.807993)
+		(start 141.629295 141.00618)
+		(end 135.69116 141.00618)
 		(width 0.5)
 		(layer "F.Cu")
@@
 	)
 	(segment
-		(start 163.216966 132.807993)
-		(end 159.035346 132.807993)
+		(start 135.69116 141.00618)
+		(end 110.501159 115.816179)
 		(width 0.5)
 		(layer "F.Cu")
@@
 	)
 	(segment
-		(start 159.035346 132.807993)
-		(end 152.650159 139.19318)
+		(start 148.977209 143.221993)
+		(end 143.845109 143.221993)
 		(width 0.5)
 		(layer "F.Cu")
@@
 	)
 	(segment
-		(start 133.878159 139.19318)
-		(end 110.501159 115.816179)
+		(start 106.44658 102.958988)
+		(end 100.189616 102.958988)
 		(width 0.5)
 		(layer "F.Cu")
@@
 	)
 	(segment
-		(start 110.501159 107.013567)
-		(end 106.44658 102.958988)
+		(start 169.398159 133.061993)
+		(end 163.470966 133.061993)
 		(width 0.5)
 		(layer "F.Cu")
@@
 	)
 	(segment
-		(start 106.44658 102.958988)
-		(end 100.189616 102.958988)
+		(start 143.845109 143.221993)
+		(end 141.629295 141.00618)
+		(width 0.5)
+		(layer "F.Cu")
+		(net "Net-(Q301-B)")
+	)
+	(segment
+		(start 110.501159 115.816179)
+		(end 110.501159 107.013567)
 		(width 0.5)
 		(layer "F.Cu")
@@
 	)
 	(segment
-		(start 152.650159 139.19318)
-		(end 133.878159 139.19318)
+		(start 163.470966 133.061993)
+		(end 163.216966 132.807993)
+		(width 0.5)
+		(layer "F.Cu")
+		(net "Net-(Q301-B)")
+	)
+	(segment
+		(start 110.501159 107.013567)
+		(end 106.44658 102.958988)
 		(width 0.5)
 		(layer "F.Cu")
@@
 	)
 	(segment
+		(start 169.782462 122.22418)
+		(end 172.707462 125.14918)
+		(width 1.25)
+		(layer "B.Cu")
+		(net "Net-(J401-Pin_2)")
+	)
+	(segment
+		(start 171.682462 117.98818)
+		(end 171.682462 120.15218)
+		(width 1.25)
+		(layer "B.Cu")
+		(net "Net-(J401-Pin_2)")
+	)
+	(segment
+		(start 172.707462 125.14918)
+		(end 172.707462 126.38218)
+		(width 1.25)
+		(layer "B.Cu")
+		(net "Net-(J401-Pin_2)")
+	)
+	(segment
+		(start 172.700159 142.110466)
+		(end 176.256159 145.666466)
+		(width 1.25)
+		(layer "B.Cu")
+		(net "Net-(J401-Pin_2)")
+	)
+	(segment
+		(start 172.707462 126.59918)
+		(end 172.707462 139.062466)
+		(width 1.25)
+		(layer "B.Cu")
+		(net "Net-(J401-Pin_2)")
+	)
+	(segment
+		(start 171.682462 120.15218)
+		(end 169.782462 122.05218)
+		(width 1.25)
+		(layer "B.Cu")
+		(net "Net-(J401-Pin_2)")
+	)
+	(segment
+		(start 172.700159 139.069769)
+		(end 172.700159 142.110466)
+		(width 1.25)
+		(layer "B.Cu")
+		(net "Net-(J401-Pin_2)")
+	)
+	(segment
+		(start 169.782462 122.05218)
+		(end 169.782462 122.22418)
+		(width 1.25)
+		(layer "B.Cu")
+		(net "Net-(J401-Pin_2)")
+	)
+	(segment
+		(start 172.707462 138.089163)
+		(end 172.707462 139.062466)
+		(width 1.25)
+		(layer "B.Cu")
+		(net "Net-(J401-Pin_2)")
+	)
+	(segment
