File: kicad/apple2-luggable-crt.kicad_sch (KiCad schematic)
At the start: 236 parts, among them J1 VIDEO IN, J401 DEFLECTION YOKE, J402 CRT SOCKET BRD, J501 CRT SOCKET BRD, J801 12V UNREG, K6 Jumper_2_Bridged, K9+ Jumper_2_Bridged, K9- Jumper_2_Bridged, Q201 2SA562-Y, Q202 2SC1815-Y, Q301 2SC2236A-Y, Q302 2SC2236A-Y, Q303 2SC1815-Y, Q304 2SA1015-Y, Q401 2SC200-Y, Q402 2SC2233, Q501 TD7698AP, Q801 PNP, SW201 SW_SP3T, SW801 SW_SPST, T401 L_Ferrite_Coupled_1243, T451 KFB-2007 / 8D04K, T502 KRFE204, X501 3.579545MHz

Commit message: more progress
Parts:
- added TP1: GND, TestPoint:TestPoint_THTPad_D3.0mm_Drill1.5mm, symbol Connector:TestPoint
- added TP41: PIN 5, TestPoint:TestPoint_THTPad_D3.0mm_Drill1.5mm, symbol Connector:TestPoint
- added TP42: PIN 8, TestPoint:TestPoint_THTPad_D3.0mm_Drill1.5mm, symbol Connector:TestPoint
- added TP43: PIN 18, TestPoint:TestPoint_THTPad_D3.0mm_Drill1.5mm, symbol Connector:TestPoint
- added TP44: PIN 13, TestPoint:TestPoint_THTPad_D3.0mm_Drill1.5mm, symbol Connector:TestPoint
- C202, C203, C206, C207, C301, C302, C304, C307, C312, C402, C403, C404, C405, C406, C407, C413, C414, C415, C417, C418, C426, C427, C428, C430, C434, C435, C501, C502, C504, C505, C506, C507, C509, C510, C511, C514, C515, C516, C517, C518: footprint (none) -> Capacitor_SMD:C_0805_2012Metric_Pad1.18x1.45mm_HandSolder
- C429: value 2.2nF -> 2.2nF 500V; footprint (none) -> Capacitor_SMD:C_0805_2012Metric_Pad1.18x1.45mm_HandSolder
- J401: footprint (none) -> foodprints:DEFLECTION_CONNECTOR
- Q801: value PNP -> 2SB953
- R202, R203, R204, R205, R206, R207, R208, R209, R210, R213, R214, R215, R218, R219, R220, R221, R222, R223, R224, R225, R226, R227, R229, R230, R301, R302, R303, R304, R305, R306, R308, R310, R312, R313, R315, R316, R317, R319, R321, R323, R324, R325, R326, R327, R328, R329, R354, R355, R401, R402, R403, R404, R405, R406, R407, R408, R409, R410, R412, R413, R414, R415, R416, R417, R419, R421, R424, R426, R501, R502, R503, R504, R507, R508, R509, R511, R512, R515, R516, R517, R518, R519, R520, R521, R522, R523, R524, R525, R526, R527, R528, R529, R530, R531, R535, RV14: footprint (none) -> Resistor_SMD:R_1206_3216Metric_Pad1.30x1.75mm_HandSolder
- R300: renamed from R??; footprint (none) -> Resistor_SMD:R_1206_3216Metric_Pad1.30x1.75mm_HandSolder
- R320: value 6.8Ω 1/2W -> 6.8Ω 1/4W
- T451: footprint (none) -> foodprints:Flyback
- T502: footprint (none) -> foodprints:CHROMA_FILTER
- TP33: value ?? -> PIN 37; footprint (none) -> TestPoint:TestPoint_THTPad_D3.0mm_Drill1.5mm
- renumbered K9+ to JPK9+1, K9- to JPK9-1, U to JPU1
Connections:
- net CHROMA: now also TP41.1
- net GNDPWR: now also T502.3, T502.4, T502.5, T502.SHIELD, TP1.1
- net at C505.2, Q501.8 (CHROMA_OUT), R511.1: now also TP42.1
- net at C515.1, Q501.18 (AFC_FILTER_2), R520.2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: now also TP43.1
- net at Q501.13 (XTAL_DRIVE), R516.1: now also TP44.1
- net HORIZ RETRACE BLANKING renamed HORIZ BLANKING
- net V SIZE renamed VERT SIZE
- net VERT RETRACE BLANKING renamed VERT BLANKING
Other:
- note added: "R300 = BOARD MOD"
- note removed: "RESISTOR WAS BOARD MOD"
- moved on the sheet: C308, C310, C312, C314, C414, C424, C513, C514, C515, D402, J401, JPU1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

Commit message: more progress
Parts:
- C201: footprint (none) -> Capacitor_THT:CP_Radial_D5.0mm_P2.00mm
- C204, C209, C210, C309, C310, C313, C412, C423, C803: footprint (none) -> Capacitor_THT:CP_Radial_D8.0mm_P3.50mm
- C205, C208, C303, C305, C308, C311, C314, C401, C408, C409, C416, C503, C508, C513, C519: footprint (none) -> Capacitor_SMD:C_0805_2012Metric_Pad1.18x1.45mm_HandSolder
- C306, C422, C424: footprint (none) -> Capacitor_THT:CP_Radial_D6.3mm_P2.50mm
- C419, C420, C421: footprint (none) -> Capacitor_THT:C_Rect_L10.3mm_W4.5mm_P7.50mm_MKS4
- D202, D203, D301, D302, D401, D402, D403: footprint (none) -> Diode_SMD:D_MiniMELF_Handsoldering
- D303: value 1SR35-100A (??) -> 1N4935; footprint (none) -> Diode_THT:D_DO-41_SOD81_P10.16mm_Horizontal
- D404: value TVR06D -> 1N4935; footprint (none) -> Diode_THT:D_DO-41_SOD81_P10.16mm_Horizontal
- D405: footprint (none) -> Diode_THT:D_DO-41_SOD81_P10.16mm_Horizontal
- D408: value RGP10G -> 1N4935; footprint (none) -> Diode_THT:D_DO-41_SOD81_P10.16mm_Horizontal
- J402: footprint (none) -> Connector_JST:JST_XH_B4B-XH-A_1x04_P2.50mm_Vertical
- J501: footprint (none) -> Connector_JST:JST_XH_B5B-XH-A_1x05_P2.50mm_Vertical
- L301: footprint Inductor_THT:L_Radial_D7.5mm_P5.00mm_Fastron_07P -> Inductor_SMD:L_1008_2520Metric_Pad1.43x2.20mm_HandSolder
- L405: footprint (none) -> foodprints:L_Radial_D10.0mm_P7.62mm
- L408, L501: footprint Inductor_THT:L_Radial_D7.5mm_P5.00mm_Fastron_07P -> Inductor_SMD:L_TDK_NLV32_3.2x2.5mm
- Q201, Q304: footprint (none) -> Package_TO_SOT_THT:TO-92_Inline_Wide; symbol Simulation_SPICE:PNP -> Transistor_BJT:Q_PNP_ECB
- Q202, Q301, Q302, Q303, Q401: footprint (none) -> Package_TO_SOT_THT:TO-92_Inline_Wide; symbol Simulation_SPICE:NPN -> Transistor_BJT:Q_NPN_ECB
- R206: value 830Ω -> 820Ω
- R321: value 160Ω 1/2 W -> 160Ω 1/2W
Connections:
- net +10V: now also Q202.2 (C); no longer Q202.1 (C)
- net +11V: now also Q304.1 (E); no longer Q304.3 (E)
- net GNDPWR: now also Q301.1 (E), Q303.1 (E); no longer Q301.3 (E), Q303.3 (E)
- net H DRIVE: now also Q401.3 (B); no longer Q401.2 (B)
- net VERT BLANKING: now also Q304.2 (C); no longer Q304.1 (C)
- net at C207.1, D203.2 (A), D301.1 (K)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: now also Q201.3 (B); no longer Q201.2 (B)
- net at Q201.1 (E): now also R222.1, SW201.3; no longer R223.2
- net at C312.1, D302.1 (K), R314.2: now also Q301.2 (C); no longer Q301.1 (C)
- net at C312.2, R310.2: now also Q301.3 (B); no longer Q301.2 (B)
- net at DL201.3, R208.1: now also Q202.3 (B); no longer Q202.2 (B)
- net at R324.2, R325.1: now also Q303.3 (B); no longer Q303.2 (B)
- net at C417.1, R417.2, T401.1: now also Q401.2 (C); no longer Q401.1 (C)
- net at L410.1: now also Q401.1 (E); no longer Q401.3 (E)
- net at C313.1, D303.1 (K): now also Q302.2 (C); no longer Q302.1 (C)
- net at C306.2, C307.1, C311.1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: now also Q302.1 (E); no longer Q302.3 (E)
- net at C205.1, R224.1: now also Q202.1 (E); no longer Q202.3 (E)
- net at D302.2 (A), R313.2: now also Q302.3 (B); no longer Q302.2 (B)
- net at R326.1: now also Q303.2 (C); no longer Q303.1 (C)
- net at R326.2, R327.2: now also Q304.3 (B); no longer Q304.2 (B)
- new net: Q201.2 (C), R223.2
Other:
- note removed: "NOTE: ERROR? SHORT TO +10?"
- moved on the sheet: C207, C414, C417, C418, C502, C514, C515, D203, D301, D402, D403, Q201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

Commit message: more work
Parts:
- added H1, H2, H3, H4, H5, H6: MountingHole_Pad, MountingHole:MountingHole_3.2mm_M3_Pad_TopBottom, symbol Mechanical:MountingHole_Pad
- added U1: MIC29302WU, Package_TO_SOT_SMD:TO-263-5_TabPin3, symbol Regulator_Linear:MIC29302WU
- R254, R255, R451, R554, R555: footprint (none) -> Potentiometer_THT:Potentiometer_Alpha_RD901F-40-00D_Single_Vertical_CircularHoles
- R257, R352, R353: footprint (none) -> Potentiometer_THT:Potentiometer_Bourns_3386F_Vertical
Connections:
- net +VCC_{H}: now also R412.1; no longer R412.2
- net GNDPWR: now also C407.1, H1.1, H2.1, H3.1, H4.1, H5.1, H6.1, U1.3 (GND); no longer C407.2
- net at C301.1, R301.2, R302.1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: now also L301.1; no longer L301.2
- net at R324.1: now also Q303.3 (B), R325.1; no longer C311.2
- net at R451.2: now also R410.1; no longer R410.2
- net at Q501.36 (SYNC_SEP._OUT), R304.2: now also L301.2; no longer L301.1
- new net: C311.2, R324.2
- new net: C407.2, Q501.34 (H_OSC_TIMING), R409.1, R410.2, R412.2
Other:
- moved on the sheet: C306, C307, C308, C309, C310, C311, C312, C313, C314, C424, C430, C803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
