File: kicad/apple2-luggable-crt.kicad_sch (KiCad schematic)
At the start: 248 parts, among them J1 VIDEO IN, J401 DEFLECTION YOKE, J402 CRT SOCKET BRD, J501 CRT SOCKET BRD, J801 12V UNREG, K6 Jumper_2_Bridged, Q201 2SA562-Y, Q202 2SC1815-Y, Q301 2SC2236A-Y, Q302 2SC2236A-Y, Q303 2SC1815-Y, Q304 2SA1015-Y, Q401 2SC200-Y, Q402 2SC2233, Q501 TD7698AP, Q801 2SB953, SW201 SW_SP3T, SW801 SW_SPST, T401 L_Ferrite_Coupled_1243, T451 KFB-2007 / 8D04K, T502 KRFE204, U1 MIC29302WU, X501 3.579545MHz

Commit message: more progress
- pretty close to being done.  now comparing foot prints to parts samples, checking part placement for interference, and making layout adjustments to accommodate PCB mounting holes now that I know where they are.
Parts:
- removed C803: 330μF 16V, Capacitor_THT:CP_Radial_D8.0mm_P3.50mm, symbol Device:C_Polarized_Small_US
- removed C9: 4700μF 16V, symbol Device:C_Polarized_Small_US
- removed F802: 125V, 2A, symbol Device:Fuse
- removed J801: 12V UNREG, Connector_BarrelJack:BarrelJack_Wuerth_6941xx301002, symbol Connector:Barrel_Jack_MountingPin
- removed JPK9+1, JPK9-1, JPU1, K6: Jumper_2_Bridged, symbol Jumper:Jumper_2_Bridged
- removed Q801: 2SB953, symbol Simulation_SPICE:PNP
- removed SW801: SW_SPST, symbol Switch:SW_SPST
- added J403, J404: PICTURE CONTROLS, Connector_JST:JST_PH_B9B-PH-K_1x09_P2.00mm_Vertical, symbol Connector_Generic:Conn_01x09
- added J801: 12V UNREG, TerminalBlock_TE-Connectivity:TerminalBlock_TE_282834-2_1x02_P2.54mm_Horizontal, symbol Connector:Screw_Terminal_01x02
- added R211: 6.81kΩ 1%, Resistor_SMD:R_1206_3216Metric_Pad1.30x1.75mm_HandSolder, symbol Device:R_Small_US
- added R212: 53.6kΩ 1%, Resistor_SMD:R_1206_3216Metric_Pad1.30x1.75mm_HandSolder, symbol Device:R_Small_US
- H1, H2, H3, H4, H5, H6: value MountingHole_Pad -> M3
- J1: footprint (none) -> Connector_Coaxial:BNC_TEConnectivity_1478204_Vertical
- R254: Comment (none) -> CONTRAST
- R255: Comment (none) -> BRIGHT
- R257: Comment (none) -> SUB BRIGHT
- R351: footprint (none) -> Potentiometer_THT:Potentiometer_Alpha_RD901F-40-00D_Single_Vertical_CircularHoles; Comment (none) -> V HOLD
- R352: Comment (none) -> V HEIGHT
- R353: Comment (none) -> V CENTRE
- R451: Comment (none) -> H HOLD
- R554: Comment (none) -> TINT
- R555: Comment (none) -> COLOUR
- U1: value MIC29302WU -> XRP29302ETBTR-L
Connections:
- net +10V: now also J403.2 (Pin_2), J404.2 (Pin_2)
- net +11V: now also U1.4 (VOUT), R212.1
- net +VCC_{H}: now also R451.1, J403.8 (Pin_8), J404.8 (Pin_8); no longer R451.3
- net COLOUR: now also J403.4 (Pin_4), J404.4 (Pin_4)
- net CONTRAST: now also J403.3 (Pin_3), J404.3 (Pin_3)
- net GNDPWR: now also R451.3, J403.5 (Pin_5), J404.5 (Pin_5), J801.2 (Pin_2), R211.2; no longer R451.1
- net TINT: now also J403.6 (Pin_6), J404.6 (Pin_6)
- net at R230.1: now also R257.3
- net BRIGHT: now reaches Q501.4 (BRIGHTNESS_CONTROL), R209.2, R219.1, R225.2
- net BRIGHT: now also J403.7 (Pin_7), J404.7 (Pin_7)
- net at R215.1, R218.2: now also R255.1; no longer R255.3
- net at R215.2, R229.1: now also R255.3; no longer R255.1
- net H HOLD: now reaches R410.1, R451.2
- net H HOLD: now also J403.9 (Pin_9), J404.9 (Pin_9)
- net at R554.1: now also R512.2; no longer R515.1
- net at R554.3: now also R515.1; no longer R512.2
- net at C415.1, R419.1, R421.2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: now also T451.
- net V HOLD: now reaches C304.1, Q501.29 (V_OSC_TIMING), R351.1, SW201.2, SW201.4
- net V HOLD: now also J403.1 (Pin_1), J404.1 (Pin_1)
- net at R504.2, R508.2, R519.1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: now also R555.1; no longer R555.3
- net at R507.1: now also R555.3; no longer R555.1
- net at U1.1 (EN): now also U1.2 (VIN), J801.1 (Pin_1)
- net at U1.5 (ADJ): now also R211.1, R212.2
- net at R254.1: now also R210.2; no longer R213.1
- net at R254.3: now also R213.1; no longer R210.2
Other:
- moved on the sheet: C301, C302, C303, C404, C405, C406, C407, C408, C409, C413, C434, C435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

Commit message: version before heat sink work
Parts:
- added HS1: Heatsink_Pad_2Pin, symbol Mechanical:Heatsink_Pad_2Pin
- added J2: FOC. SCN. RET., Connector_PinHeader_2.54mm:PinHeader_1x01_P2.54mm_Vertical, symbol Connector_Generic:Conn_01x01
- H1, H2, H3, H4: value M3 -> M4; footprint MountingHole:MountingHole_3.2mm_M3_Pad_TopBottom -> MountingHole:MountingHole_4.3mm_M4_Pad_TopBottom
- H5, H6: footprint MountingHole:MountingHole_3.2mm_M3_Pad_TopBottom -> foodprints:MountingHole_3.2mm_M3_Pad_TopBottom_flyback_shield
- J801: footprint TerminalBlock_TE-Connectivity:TerminalBlock_TE_282834-2_1x02_P2.54mm_Horizontal -> Connector_JST:JST_VH_B2P-VH_1x02_P3.96mm_Vertical
- renumbered RV14 to R129
Connections:
- net GNDPWR: now also HS1.1, HS1.2
- net 12 V UNREG: now reaches J801.1 (Pin_1), U1.1 (EN), U1.2 (VIN)
- net at C415.1, R419.1, R421.2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: now also J2.1 (Pin_1)
- net HEATER ACV: now reaches J402.1 (Pin_1), L403.2
- net 90V: now reaches C422.1, D405.1 (K), J402.4 (Pin_4), R425.1
Other:
- note added: "BOARD MOUNTING HOLES"
- note added: "MOUNTING HOLES FOR FLYBACK SHIELD"
- moved on the sheet: H5, H6, J801

Commit message: finished.
Parts:
- HS1: footprint (none) -> foodprints:Heatsink_TO-220_26x20mm_2xFixation1.2mm
Changed lines of the file:
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@@
 			)
 		)
-		(property "Footprint" ""
+		(property "Footprint" "foodprints:Heatsink_TO-220_26x20mm_2xFixation1.2mm"
 			(at 185.7248 234.95 0)
 			(hide yes)
